File: hardware/VIP.brd (EAGLE design)
At the start: 49 x 31 mm, 29 parts, among them J1 CON254_2WAY

Commit message: Add files via upload
Parts:
- added ISP: CON254_6WAY254-2X3, Connectors:CON254MM08_2X3
- moved C7 1.71 mm to (60.6, 53.8)
- moved OP2340\ 1.02 mm to (56.6, 55.1)
- moved R6 0.40 mm to (43.3, 63.4)
- moved R5 0.40 mm to (43.3, 65.2)
Connections:
- removed net N$12: TINY841.P$10, U$1.P$2
- removed net N$14: TINY841.P$8, U$1.P$4
- removed net N$15: TINY841.P$7, U$1.P$5
- new net MISO: ISP.P$1, TINY841.P$13, U$1.P$1
- new net MOSI: ISP.P$4, TINY841.P$12, U$1.P$2
- new net RESET: ISP.P$5, TINY841.P$4
- new net SCK: ISP.P$3, TINY841.P$10
- net GND: now also ISP.P$6
- net IMEASURE: now also TINY841.P$8; no longer TINY841.P$13
- net N$10: no longer U$1.P$1
- net N$13: no longer U$1.P$3
- net VCC: now also ISP.P$2
- net VMEASURE: now also TINY841.P$7; no longer TINY841.P$12
Routing:
- net RESET: track 0.00 -> 59.2 mm, vias 0 -> 2
- net MOSI: track 0.00 -> 41.8 mm, vias 0 -> 1
- net N$15: track 36.6 -> 0.00 mm
- net MISO: track 0.00 -> 28.8 mm
- net SCK: track 0.00 -> 28.1 mm, vias 0 -> 1
- net N$10: track 27.4 -> 0.00 mm
- net N$12: track 26.4 -> 0.00 mm
- net N$13: track 25.5 -> 0.00 mm
- net N$14: track 25.0 -> 0.00 mm
- net VMEASURE: track 11.1 -> 25.8 mm, vias 0 -> 2
- net IMEASURE: track 11.9 -> 19.0 mm, vias 0 -> 2
- net VCC: track 98.7 -> 103.5 mm
- net V+: track 62.6 -> 60.6 mm
- net N$16: track 36.1 -> 37.2 mm, vias 0 -> 2
- net N$3: track 19.1 -> 20.2 mm
Other:
- board text added: "ISP"

Commit message: Add files via upload
Parts:
- removed J1: CON254_2WAY, Connectors:CON254MM08_1X2
- removed R1, R2: 25k, rcl:M0805
- removed R3, R4, R7, R8: 10k, rcl:M0805
- removed R5, R6: 25k, RLC:0603L
- removed U$1: CON254_8WAY, Connectors:CON254MM08_1X6
- added J2: CON254_18WAY3X6, Connectors:CON254MM08_3X6
- added R10, R15, R9: 10k, RLC:0603L
- added R11, R12, R13, R14: 25k, RLC:0603L
- added R16: 150k, RLC:0603L
- ISP: value CON254_6WAY254-2X3 -> CON254_6WAY254-2X3-EDGE; device Connectors:CON254MM08_2X3 -> Connectors:CON254MM08_2X3_EDGE
- moved TINY841 16.1 mm to (59.6, 57.7), turned to 90 degrees
- moved OP2340\ 13.5 mm to (43.2, 53.4)
- moved ISP 9.92 mm to (71.4, 69.6), turned to 0 degrees
- moved C2 5.92 mm to (49.8, 55.4)
- moved C4 4.00 mm to (36.6, 55.7), turned to 90 degrees
- moved C7 3.04 mm to (60.5, 56.8), turned to 45 degrees
- moved D1 2.69 mm to (42.6, 52.9)
- moved L1 2.50 mm to (49.0, 52.9)
- moved MAX5035 2.50 mm to (46.4, 61.7)
- moved C5 1.18 mm to (38.5, 55.7), turned to 90 degrees
- moved C1 0.11 mm to (40.5, 62.0), turned to 90 degrees
Connections:
- net GND: now also J2.P$1, J2.P$2, J2.P$3, J2.P$4, J2.P$5, J2.P$6, R10.P$2, R11.P$2, R12.P$2, R14.P$2, R15.P$2; no longer J1.P$1, R1.1, R2.1, R3.1, R5.P$1, R7.1
- net MISO: now also J2.P$7; no longer U$1.P$1
- net MOSI: now also J2.P$8; no longer U$1.P$2
- net N$1: now also R12.P$1, R13.P$2; no longer R5.P$2, R6.P$1
- net N$10: now also J2.P$9
- net N$11: now also R15.P$1, R16.P$2; no longer R7.2, R8.1
- net N$13: now also J2.P$11
- net N$16: now also J2.P$12; no longer U$1.P$6
- net N$3: now also R14.P$1; no longer R2.2
- net N$4: now also R11.P$1; no longer R1.2
- net N$5: now also R10.P$1, R9.P$2; no longer R3.2, R4.1
- net SCK: now also J2.P$10
- net V+: now also R13.P$1, R16.P$1; no longer R6.P$2, R8.2
- net VCC: now also J2.P$13, J2.P$14, J2.P$15, J2.P$16, J2.P$17, J2.P$18, R9.P$1; no longer J1.P$2, R4.2
Routing:
- net TOBLE: track 10.7 -> 35.8 mm
- net TOAT: track 13.2 -> 37.8 mm
- net RESET: track 59.2 -> 36.8 mm, vias 2 -> 3
- net VCC: track 103.5 -> 121.7 mm, vias 4 -> 5
- net N$16: track 37.2 -> 19.0 mm
- net N$10: track 0.00 -> 15.3 mm
- net MISO: track 28.8 -> 42.0 mm, vias 0 -> 2
- net N$13: track 0.00 -> 11.5 mm
- net IMEASURE: track 19.0 -> 30.1 mm
- net N$3: track 20.2 -> 11.9 mm
- net VMEASURE: track 25.8 -> 33.2 mm
- net N$11: track 16.1 -> 9.79 mm, vias 2 -> 0
- net MOSI: track 41.8 -> 37.1 mm
- net N$6: track 4.95 -> 9.34 mm
- net GND: track 3.06 -> 0.00 mm, vias 36 -> 18
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Other:
- board size 49 x 31 mm -> 54.6 x 28 mm

Commit message: Add files via upload
Parts:
- added D2: SINGLELEDKP-3216SRC-PRV, OptoElectronics:LED3.2X1.6MM
- added R1: 300, RLC:0603L
- added SW1: SWITCH-1P2T, Switches:JS102011
- moved C6 5.49 mm to (36.0, 52.6), turned to 45 degrees
- moved C2 4.15 mm to (46.2, 53.4), turned to 270 degrees
- moved C5 2.42 mm to (38.6, 58.1)
- moved C4 2.41 mm to (36.6, 58.1)
- moved R16 1.80 mm to (49.8, 53.6)
- moved R14 1.80 mm to (49.8, 55.4)
- moved R15 1.80 mm to (49.8, 51.8)
Connections:
- new net N$12: C6.P$1, L1.P$2, MAX5035.P$4, SW1.P$2
- new net N$14: D2.P$1, R1.P$2
- net GND: now also D2.P$2
- net VCC: now also R1.P$1, SW1.P$3; no longer C6.P$1, L1.P$2, MAX5035.P$4
Routing:
- net N$12: track 0.00 -> 39.4 mm, vias 0 -> 2
- net RESET: track 36.8 -> 24.5 mm, vias 3 -> 2
- net VCC: track 121.7 -> 116.7 mm, vias 5 -> 10
- net VMEASURE: track 33.2 -> 28.9 mm
- net N$14: track 0.00 -> 3.08 mm
- net V+: track 61.7 -> 59.9 mm
- net N$9: track 7.13 -> 5.34 mm
- net N$11: track 9.79 -> 11.4 mm
- net N$6: track 9.34 -> 7.80 mm
- net MOSI: track 37.1 -> 36.0 mm
- net SCK: track 27.0 -> 28.0 mm
- net N$8: track 18.2 -> 19.1 mm
- net MISO: track 42.0 -> 42.8 mm
Other:
- board text added: "GNDbat"
- board text added: "GNDesc"
- board text added: "Vbat"
- board text added: "Vesc"
- board text removed: "5V"
- board text removed: "A1"
- board text removed: "A2"
- board text removed: "A3"
- board text removed: "A4"
- board text removed: "A5"
- board text removed: "A6"
- board text removed: "GND"
- board text removed: "ISP"

Commit message: Add files via upload
Routing:
- net VMEASURE: track 28.9 -> 27.1 mm
Changed lines of the file:
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@@
 <setting verticaltext="up"/>
 </settings>
-<grid distance="0.014" unitdist="mm" unit="mm" style="dots" multiple="1" display="yes" altdistance="0.025" altunitdist="inch" altunit="inch"/>
+<grid distance="0.1" unitdist="mm" unit="mm" style="dots" multiple="1" display="yes" altdistance="0.025" altunitdist="inch" altunit="inch"/>
 <layers>
 <layer number="1" name="Top" color="4" fill="1" visible="yes" active="yes"/>
 <layer number="16" name="Bottom" color="1" fill="1" visible="yes" active="yes"/>
-<layer number="17" name="Pads" color="2" fill="1" visible="no" active="yes"/>
-<layer number="18" name="Vias" color="2" fill="1" visible="no" active="yes"/>
-<layer number="19" name="Unrouted" color="6" fill="1" visible="no" active="yes"/>
+<layer number="17" name="Pads" color="2" fill="1" visible="yes" active="yes"/>
+<layer number="18" name="Vias" color="2" fill="1" visible="yes" active="yes"/>
+<layer number="19" name="Unrouted" color="6" fill="1" visible="yes" active="yes"/>
 <layer number="20" name="Dimension" color="15" fill="1" visible="yes" active="yes"/>
 <layer number="21" name="tPlace" color="7" fill="1" visible="yes" active="yes"/>
@@
 <via x="63.3" y="51.7" extent="1-16" drill="0.3"/>
 <contactref element="D2" pad="P$2"/>
-<via x="42.19" y="57.014" extent="1-16" drill="0.3"/>
+<via x="42.182" y="57.056" extent="1-16" drill="0.3"/>
 <via x="40.285" y="57.522" extent="1-16" drill="0.3"/>
 <via x="45.229" y="64.051" extent="1-16" drill="0.3"/>
@@
 <wire x1="50.2" y1="65.2" x2="50.435" y2="64.965" width="0.3048" layer="1"/>
 <wire x1="50.435" y1="64.965" x2="50.435" y2="64.4" width="0.3048" layer="1"/>
-<wire x1="41.6" y1="58.2" x2="41.619" y2="58.2" width="0.3048" layer="1"/>
-<via x="41.619" y="58.2" extent="1-16" drill="0.3"/>
+<wire x1="41.6" y1="58.2" x2="41.519" y2="58.2" width="0.3048" layer="1"/>
+<via x="41.519" y="58.2" extent="1-16" drill="0.3"/>
 <wire x1="44.1548" y1="59.8028" x2="44.1548" y2="58.2" width="0.3048" layer="1"/>
 <via x="44.1548" y="58.2" extent="1-16" drill="0.3"/>
-<wire x1="44.1548" y1="58.2" x2="41.619" y2="58.2" width="0.3048" layer="16"/>
+<wire x1="44.1548" y1="58.2" x2="41.519" y2="58.2" width="0.3048" layer="16"/>
 <wire x1="44.1548" y1="52.1548" x2="44.765" y2="52.765" width="0.3048" layer="1"/>
 <wire x1="44.765" y1="52.765" x2="46.1798" y2="52.765" width="0.3048" layer="1"/>
@@
 <wire x1="40.513" y1="62.592" x2="40.52" y2="62.585" width="0.4064" layer="1"/>
 <via x="44.765" y="52.765" extent="1-16" drill="0.3"/>
-<wire x1="44.765" y1="52.765" x2="43.682" y2="53.848" width="0.254" layer="1"/>
-<wire x1="43.682" y1="53.848" x2="42.291" y2="53.848" width="0.254" layer="1"/>
-<wire x1="42.291" y1="53.848" x2="41.275" y2="54.864" width="0.254" layer="1"/>
-<wire x1="41.275" y1="54.864" x2="41.275" y2="57.15" width="0.254" layer="1"/>
-<wire x1="41.275" y1="57.15" x2="41.619" y2="57.494" width="0.254" layer="1"/>
-<wire x1="41.619" y1="57.494" x2="41.619" y2="58.2" width="0.254" layer="1"/>
+<wire x1="44.765" y1="52.765" x2="43.882" y2="53.648" width="0.254" layer="1"/>
+<wire x1="43.882" y1="53.648" x2="42.491" y2="53.648" width="0.254" layer="1"/>
 <wire x1="44.765" y1="52.765" x2="52.518" y2="52.765" width="0.3048" layer="16"/>
 <wire x1="52.518" y1="52.765" x2="53.213" y2="52.07" width="0.3048" layer="16"/>
@@
 <wire x1="41.656" y1="62.585" x2="38.885" y2="62.585" width="0.3048" layer="16"/>
 <wire x1="38.885" y1="62.585" x2="38.05" y2="61.75" width="0.3048" layer="16"/>
-<wire x1="41.656" y1="62.585" x2="41.656" y2="58.237" width="0.3048" layer="1"/>
-<wire x1="41.656" y1="58.237" x2="41.619" y2="58.2" width="0.3048" layer="1"/>
+<wire x1="41.656" y1="62.585" x2="41.656" y2="58.337" width="0.3048" layer="1"/>
+<wire x1="41.656" y1="58.337" x2="41.519" y2="58.2" width="0.3048" layer="1"/>
+<wire x1="41.519" y1="58.2" x2="41.519" y2="54.62" width="0.254" layer="1"/>
+<wire x1="41.519" y1="54.62" x2="42.491" y2="53.648" width="0.254" layer="1"/>
 </signal>
 <signal name="IMEASURE">
@@
 <wire x1="49.165" y1="60.8" x2="49.165" y2="59" width="0.3048" layer="1"/>
 <wire x1="49.165" y1="60.8" x2="47.8" y2="60.8" width="0.3048" layer="1"/>
-<wire x1="47.8" y1="60.8" x2="47.2" y2="61.4" width="0.3048" layer="1"/>
-<via x="47.2" y="61.4" extent="1-16" drill="0.3"/>
-<wire x1="47.2" y1="61.4" x2="47.2" y2="63" width="0.3048" layer="16"/>
+<via x="47.2" y="62.2" extent="1-16" drill="0.3"/>
+<wire x1="47.2" y1="62.2" x2="47.2" y2="63" width="0.3048" layer="16"/>
 <wire x1="47.2" y1="63" x2="47.8" y2="63.6" width="0.3048" layer="16"/>
 <wire x1="47.8" y1="63.6" x2="49.316" y2="63.6" width="0.3048" layer="16"/>
 <wire x1="49.316" y1="63.6" x2="49.321" y2="63.605" width="0.3048" layer="16"/>
+<wire x1="47.2" y1="62.2" x2="47.2" y2="61.4" width="0.254" layer="1"/>
+<wire x1="47.2" y1="61.4" x2="47.8" y2="60.8" width="0.254" layer="1"/>
 </signal>
 <signal name="N$8">
@@
 <wire x1="62.7" y1="55.9" x2="63.41" y2="55.19" width="0.254" layer="1"/>
 <wire x1="63.41" y1="55.19" x2="63.41" y2="54.3" width="0.254" layer="1"/>
-<wire x1="42.8548" y1="52.8452" x2="42.5" y2="53.2" width="0.254" layer="1"/>
-<wire x1="42.5" y1="53.2" x2="42" y2="53.2" width="0.254" layer="1"/>
-<via x="42" y="53.2" extent="1-16" drill="0.3"/>
-<wire x1="42" y1="53.2" x2="44.056" y2="53.2" width="0.254" layer="16"/>
-<wire x1="44.056" y1="53.2" x2="44.45" y2="53.594" width="0.254" layer="16"/>
+<wire x1="43.7012" y1="52.8452" x2="44.45" y2="53.594" width="0.254" layer="16"/>
 <wire x1="44.45" y1="53.594" x2="54.394" y2="53.594" width="0.254" layer="16"/>
+<via x="42.8548" y="52.8452" extent="1-16" drill="0.3"/>
+<wire x1="42.8548" y1="52.8452" x2="43.7012" y2="52.8452" width="0.254" layer="16"/>
 </signal>
 <signal name="N$11">

Commit message: Add files via upload
Other:
- board text added: "v1.0 protonwheels.com"
Changed lines of the file:
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@@
 <grid distance="0.1" unitdist="mm" unit="mm" style="dots" multiple="1" display="yes" altdistance="0.025" altunitdist="inch" altunit="inch"/>
 <layers>
-<layer number="1" name="Top" color="4" fill="1" visible="yes" active="yes"/>
+<layer number="1" name="Top" color="4" fill="1" visible="no" active="yes"/>
 <layer number="16" name="Bottom" color="1" fill="1" visible="yes" active="yes"/>
 <layer number="17" name="Pads" color="2" fill="1" visible="yes" active="yes"/>
@@
 <layer number="19" name="Unrouted" color="6" fill="1" visible="yes" active="yes"/>
 <layer number="20" name="Dimension" color="15" fill="1" visible="yes" active="yes"/>
-<layer number="21" name="tPlace" color="7" fill="1" visible="yes" active="yes"/>
+<layer number="21" name="tPlace" color="7" fill="1" visible="no" active="yes"/>
 <layer number="22" name="bPlace" color="7" fill="1" visible="yes" active="yes"/>
-<layer number="23" name="tOrigins" color="15" fill="1" visible="yes" active="yes"/>
+<layer number="23" name="tOrigins" color="15" fill="1" visible="no" active="yes"/>
 <layer number="24" name="bOrigins" color="15" fill="1" visible="yes" active="yes"/>
-<layer number="25" name="tNames" color="7" fill="1" visible="yes" active="yes"/>
+<layer number="25" name="tNames" color="7" fill="1" visible="no" active="yes"/>
 <layer number="26" name="bNames" color="7" fill="1" visible="yes" active="yes"/>
 <layer number="27" name="tValues" color="7" fill="1" visible="no" active="yes"/>
@@
 <layer number="98" name="Guide" color="6" fill="1" visible="no" active="no"/>
 <layer number="200" name="200bmp" color="13" fill="2" visible="yes" active="yes"/>
-<layer number="201" name="201bmp" color="2" fill="10" visible="yes" active="yes"/>
-<layer number="202" name="202bmp" color="3" fill="10" visible="yes" active="yes"/>
+<layer number="201" name="201bmp" color="2" fill="10" visible="no" active="yes"/>
+<layer number="202" name="202bmp" color="3" fill="10" visible="no" active="yes"/>
 </layers>
 <board>
@@
 <rectangle x1="62.111" y1="52.423" x2="62.167" y2="52.437" layer="200"/>
 <rectangle x1="62.671" y1="52.423" x2="62.713" y2="52.437" layer="200"/>
+<text x="67.1" y="47.8" size="1.016" layer="26" rot="MR0">v1.0
+protonwheels.com</text>
 </plain>
 <attributes>
@@
 </element>
 <element name="C3" library="RLC" package="0603L" value="0.1uF" x="34.2" y="59.9" smashed="yes" rot="MR180">
-<attribute name="NAME" x="35.73" y="59.9856" size="0.6096" layer="26" rot="MR180"/>
+<attribute name="NAME" x="32.47" y="59.8144" size="0.6096" layer="26" rot="MR0"/>
 <attribute name="VALUE" x="32.93" y="60.789" size="0.6096" layer="28" rot="MR0" align="bottom-right"/>
 </element>
@@
 </element>
 <element name="C4" library="RLC" package="0603L" value="0.1uF" x="36.64" y="58.098" smashed="yes" rot="MR90">
-<attribute name="NAME" x="36.3544" y="59.628" size="0.6096" layer="26" rot="MR90"/>
+<attribute name="NAME" x="35.5456" y="57.972" size="0.6096" layer="26" rot="MR270"/>
 <attribute name="VALUE" x="35.751" y="56.828" size="0.6096" layer="28" rot="MR270" align="bottom-right"/>
 </element>
 <element name="C5" library="RLC" package="0603L" value="0.1uF" x="38.587" y="58.098" smashed="yes" rot="MR90">
-<attribute name="NAME" x="38.2214" y="59.628" size="0.6096" layer="26" rot="MR90"/>
+<attribute name="NAME" x="39.6214" y="58.328" size="0.6096" layer="26" rot="MR90"/>
 <attribute name="VALUE" x="37.698" y="56.828" size="0.6096" layer="28" rot="MR270" align="bottom-right"/>
 </element>
 <element name="L1" library="RLC" package="SRN8040" value="100uH" x="49" y="52.9" smashed="yes" rot="MR0">
-<attribute name="NAME" x="53.3" y="48.84" size="1.27" layer="26" rot="MR180"/>
+<attribute name="NAME" x="53" y="53.34" size="1.27" layer="26" rot="MR180"/>
 <attribute name="VALUE" x="44.5" y="55.9" size="1.27" layer="28" rot="MR270"/>
 </element>
@@
 </board>
 </drawing>
+<compatibility>
+<note version="6.3" minversion="6.2.2" severity="warning">
+Since Version 6.2.2 text objects can contain more than one line,
+which will not be processed correctly with this version.
+</note>
+</compatibility>
 </eagle>

Commit message: Add files via upload
Parts:
- added R2, R3, R4, R5: 10k, RLC:0603L
- added T1: 2N7002, Semiconductors:SOT-563
- added U1: L78L33A, Power:SOT-89
- moved C4 6.49 mm to (41.7, 62.2), turned to 180 degrees
- moved R1 6.00 mm to (23.5, 64.0)
- moved SW1 5.00 mm to (23.4, 55.0)
- moved BLE14 5.00 mm to (24.8, 55.0)
- moved D2 5.00 mm to (18.9, 64.0)
- moved C6 3.94 mm to (32.8, 55.0), turned to 270 degrees
- moved C5 3.55 mm to (41.7, 59.8), turned to 180 degrees
- moved MAX5035 2.60 mm to (49.0, 61.7)
- moved C3 1.81 mm to (32.4, 59.7)
- moved C2 0.20 mm to (46.4, 53.4)
- renumbered OP2340\ to OP2340
Connections:
- removed net TOBLE: BLE14.P$4, TINY841.P$6
- new net N$17: R3.P$2, T1.P$4, TINY841.P$6
- new net N$19: BLE14.P$2, R4.P$2, T1.P$6
- new net N$21: BLE14.P$4, R2.P$2, T1.P$3
- new net V3.3: BLE14.P$9, C3.P$1, R2.P$1, R4.P$1, T1.P$2, T1.P$5, U1.P$1
- net GND: now also U1.P$2
- net TOAT: now also R5.P$2, T1.P$1; no longer BLE14.P$2
- net VCC: now also R3.P$1, R5.P$1, U1.P$3; no longer BLE14.P$9, C3.P$1
Routing:
- net N$17: track 0.00 -> 40.5 mm
- net VCC: track 116.6 -> 155.8 mm, vias 10 -> 11
- net TOBLE: track 35.3 -> 0.00 mm
- net N$19: track 0.00 -> 25.7 mm
- net V3.3: track 0.00 -> 25.2 mm, vias 0 -> 1
- net N$21: track 0.00 -> 19.9 mm
- net N$12: track 39.4 -> 50.9 mm
- net N$8: track 19.1 -> 23.8 mm
- net N$6: track 7.80 -> 4.20 mm
- net TOAT: track 37.3 -> 34.6 mm, vias 0 -> 2
- net V+: track 59.9 -> 62.0 mm
- net N$9: track 5.34 -> 3.75 mm
- net N$4: track 11.5 -> 10.3 mm, vias 0 -> 2
- net N$1: track 7.99 -> 9.08 mm
- net N$14: track 3.08 -> 2.08 mm
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Other:
- board size 54.6 x 28 mm -> 59.6 x 28 mm

Commit message: Add files via upload
Parts:
- renumbered BLE14 to BLE11

Commit message: Add files via upload
Parts:
- moved C6 0.89 mm to (32.0, 55.4), turned to 135 degrees
Connections:
- net GND: now also SW1.P$1
- net N$1: now also SW1.P$2
- net N$12: no longer SW1.P$2
- net VCC: no longer SW1.P$3
Routing:
- net N$1: track 9.08 -> 38.9 mm, vias 1 -> 3
- net N$12: track 50.9 -> 42.2 mm
- net VCC: track 155.8 -> 147.2 mm
- net V3.3: track 25.2 -> 24.2 mm
- net TOAT: track 34.6 -> 33.7 mm
