File: hardware/VIP.sch (EAGLE design)
At the start: 29 parts, among them J1 CON254_2WAY

Commit message: Add files via upload
Parts:
- added ISP: CON254_6WAY254-2X3, Connectors:CON254_6WAY254-2X3
Connections:
- removed net N$12: TINY841.PA3, U$1G$2.J$1
- removed net N$14: TINY841.PA5, U$1G$4.J$1
- removed net N$15: TINY841.PA6, U$1G$5.J$1
- new net MISO: ISP1.J$1, TINY841.PA0, U$1G$1.J$1
- new net MOSI: ISP4.J$1, TINY841.PA1, U$1G$2.J$1
- new net RESET: ISP5.J$1, TINY841.PB3
- new net SCK: ISP3.J$1, TINY841.PA3
- net GND: now also ISP6.J$1
- net IMEASURE: now also TINY841.PA5; no longer TINY841.PA0
- net N$10: no longer U$1G$1.J$1
- net N$13: no longer U$1G$3.J$1
- net VCC: now also ISP2.J$1
- net VMEASURE: now also TINY841.PA6; no longer TINY841.PA1
Other:
- moved on the sheet: U$1G$1, U$1G$2, U$1G$3, U$1G$4, U$1G$5
Changed lines of the file:
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@@
 <part name="GND16" library="supply1" deviceset="GND" device=""/>
 <part name="P+8" library="supply1" deviceset="VCC" device=""/>
+<part name="ISP" library="Connectors" deviceset="CON254_6WAY" device="254-2X3"/>
 </parts>
 <sheets>
@@
 <instance part="R8" gate="G$1" x="5.08" y="55.88" rot="R90"/>
 <instance part="V+IN3" gate="1" x="5.08" y="66.04"/>
-<instance part="U$1" gate="G$1" x="48.26" y="0" rot="R180"/>
-<instance part="U$1" gate="G$2" x="48.26" y="-2.54" rot="R180"/>
-<instance part="U$1" gate="G$3" x="48.26" y="-5.08" rot="R180"/>
-<instance part="U$1" gate="G$4" x="48.26" y="-7.62" rot="R180"/>
-<instance part="U$1" gate="G$5" x="48.26" y="-10.16" rot="R180"/>
+<instance part="U$1" gate="G$1" x="48.26" y="7.62" rot="R180"/>
+<instance part="U$1" gate="G$2" x="48.26" y="5.08" rot="R180"/>
+<instance part="U$1" gate="G$3" x="48.26" y="2.54" rot="R180"/>
+<instance part="U$1" gate="G$4" x="48.26" y="0" rot="R180"/>
+<instance part="U$1" gate="G$5" x="48.26" y="-2.54" rot="R180"/>
 <instance part="U$1" gate="G$6" x="-15.24" y="2.54"/>
 <instance part="J1" gate="G$1" x="48.26" y="-22.86" rot="R180"/>
@@
 <instance part="GND16" gate="1" x="43.18" y="-27.94"/>
 <instance part="P+8" gate="VCC" x="43.18" y="-12.7"/>
+<instance part="ISP" gate="1" x="83.82" y="53.34" rot="R180"/>
+<instance part="ISP" gate="2" x="96.52" y="53.34"/>
+<instance part="ISP" gate="3" x="83.82" y="50.8" rot="R180"/>
+<instance part="ISP" gate="4" x="96.52" y="50.8"/>
+<instance part="ISP" gate="5" x="83.82" y="48.26" rot="R180"/>
+<instance part="ISP" gate="6" x="96.52" y="48.26"/>
 </instances>
 <busses>
@@
 <wire x1="43.18" y1="-22.86" x2="43.18" y2="-25.4" width="0.1524" layer="91"/>
 </segment>
+<segment>
+<pinref part="ISP" gate="6" pin="J$1"/>
+<wire x1="99.06" y1="48.26" x2="109.22" y2="48.26" width="0.1524" layer="91"/>
+<label x="109.22" y="48.26" size="1.778" layer="95" xref="yes"/>
+</segment>
 </net>
 <net name="N$3" class="0">
@@
 <wire x1="43.18" y1="-17.78" x2="45.72" y2="-17.78" width="0.1524" layer="91"/>
 </segment>
+<segment>
+<pinref part="ISP" gate="2" pin="J$1"/>
+<wire x1="99.06" y1="53.34" x2="109.22" y2="53.34" width="0.1524" layer="91"/>
+<label x="109.22" y="53.34" size="1.778" layer="95" xref="yes"/>
+</segment>
 </net>
 <net name="IMEASURE" class="0">
@@
 </segment>
 <segment>
-<pinref part="TINY841" gate="G$1" pin="PA0"/>
-<wire x1="10.16" y1="7.62" x2="12.7" y2="7.62" width="0.1524" layer="91"/>
-<label x="12.7" y="7.62" size="1.778" layer="95" xref="yes"/>
+<pinref part="TINY841" gate="G$1" pin="PA5"/>
+<wire x1="10.16" y1="-5.08" x2="35.56" y2="-5.08" width="0.1524" layer="91"/>
+<label x="35.56" y="-5.08" size="1.778" layer="95" xref="yes"/>
 </segment>
 </net>
@@
 <net name="VMEASURE" class="0">
 <segment>
-<pinref part="TINY841" gate="G$1" pin="PA1"/>
-<wire x1="10.16" y1="5.08" x2="30.48" y2="5.08" width="0.1524" layer="91"/>
-<label x="30.48" y="5.08" size="1.778" layer="95" xref="yes"/>
-</segment>
-<segment>
 <pinref part="OP2340\" gate="G$2" pin="IN-"/>
 <wire x1="17.78" y1="43.18" x2="15.24" y2="43.18" width="0.1524" layer="91"/>
@@
 <label x="35.56" y="45.72" size="1.778" layer="95" xref="yes"/>
 </segment>
+<segment>
+<pinref part="TINY841" gate="G$1" pin="PA6"/>
+<wire x1="10.16" y1="-7.62" x2="33.02" y2="-7.62" width="0.1524" layer="91"/>
+<label x="33.02" y="-7.62" size="1.778" layer="95" xref="yes"/>
+</segment>
 </net>
 <net name="N$11" class="0">
@@
 <segment>
 <pinref part="TINY841" gate="G$1" pin="PA2"/>
-<wire x1="10.16" y1="2.54" x2="43.18" y2="2.54" width="0.1524" layer="91"/>
-<wire x1="43.18" y1="2.54" x2="43.18" y2="0" width="0.1524" layer="91"/>
-<pinref part="U$1" gate="G$1" pin="J$1"/>
-<wire x1="43.18" y1="0" x2="45.72" y2="0" width="0.1524" layer="91"/>
-</segment>
-</net>
-<net name="N$12" class="0">
-<segment>
-<pinref part="TINY841" gate="G$1" pin="PA3"/>
-<wire x1="10.16" y1="0" x2="40.64" y2="0" width="0.1524" layer="91"/>
-<wire x1="40.64" y1="0" x2="40.64" y2="-2.54" width="0.1524" layer="91"/>
-<pinref part="U$1" gate="G$2" pin="J$1"/>
-<wire x1="40.64" y1="-2.54" x2="45.72" y2="-2.54" width="0.1524" layer="91"/>
+<wire x1="10.16" y1="2.54" x2="45.72" y2="2.54" width="0.1524" layer="91"/>
 </segment>
 </net>
@@
 <segment>
 <pinref part="TINY841" gate="G$1" pin="PA4"/>
-<wire x1="10.16" y1="-2.54" x2="38.1" y2="-2.54" width="0.1524" layer="91"/>
-<wire x1="38.1" y1="-2.54" x2="38.1" y2="-5.08" width="0.1524" layer="91"/>
-<pinref part="U$1" gate="G$3" pin="J$1"/>
-<wire x1="38.1" y1="-5.08" x2="45.72" y2="-5.08" width="0.1524" layer="91"/>
-</segment>
-</net>
-<net name="N$14" class="0">
-<segment>
-<pinref part="TINY841" gate="G$1" pin="PA5"/>
-<wire x1="10.16" y1="-5.08" x2="35.56" y2="-5.08" width="0.1524" layer="91"/>
-<pinref part="U$1" gate="G$4" pin="J$1"/>
-<wire x1="35.56" y1="-5.08" x2="35.56" y2="-7.62" width="0.1524" layer="91"/>
-<wire x1="35.56" y1="-7.62" x2="45.72" y2="-7.62" width="0.1524" layer="91"/>
-</segment>
-</net>
-<net name="N$15" class="0">
-<segment>
-<pinref part="TINY841" gate="G$1" pin="PA6"/>
-<wire x1="10.16" y1="-7.62" x2="33.02" y2="-7.62" width="0.1524" layer="91"/>
-<wire x1="33.02" y1="-7.62" x2="33.02" y2="-10.16" width="0.1524" layer="91"/>
-<pinref part="U$1" gate="G$5" pin="J$1"/>
-<wire x1="33.02" y1="-10.16" x2="45.72" y2="-10.16" width="0.1524" layer="91"/>
+<wire x1="10.16" y1="-2.54" x2="45.72" y2="-2.54" width="0.1524" layer="91"/>
 </segment>
 </net>
@@
 </segment>
 </net>
+<net name="MISO" class="0">
+<segment>
+<pinref part="ISP" gate="1" pin="J$1"/>
+<wire x1="81.28" y1="53.34" x2="71.12" y2="53.34" width="0.1524" layer="91"/>
+<label x="71.12" y="53.34" size="1.778" layer="95" rot="R180" xref="yes"/>
+</segment>
+<segment>
+<pinref part="TINY841" gate="G$1" pin="PA0"/>
+<label x="22.86" y="7.62" size="1.778" layer="95" xref="yes"/>
+<pinref part="U$1" gate="G$1" pin="J$1"/>
+<wire x1="10.16" y1="7.62" x2="45.72" y2="7.62" width="0.1524" layer="91"/>
+</segment>
+</net>
+<net name="SCK" class="0">
+<segment>
+<pinref part="ISP" gate="3" pin="J$1"/>
+<wire x1="81.28" y1="50.8" x2="78.74" y2="50.8" width="0.1524" layer="91"/>
+<label x="78.74" y="50.8" size="1.778" layer="95" rot="R180" xref="yes"/>
+</segment>
+<segment>
+<pinref part="TINY841" gate="G$1" pin="PA3"/>
+<wire x1="10.16" y1="0" x2="45.72" y2="0" width="0.1524" layer="91"/>
+<label x="12.7" y="0" size="1.778" layer="95" xref="yes"/>
+</segment>
+</net>
+<net name="RESET" class="0">
+<segment>
+<pinref part="ISP" gate="5" pin="J$1"/>
+<wire x1="81.28" y1="48.26" x2="71.12" y2="48.26" width="0.1524" layer="91"/>
+<label x="71.12" y="48.26" size="1.778" layer="95" rot="R180" xref="yes"/>
+</segment>
+<segment>
+<pinref part="TINY841" gate="G$1" pin="PB3"/>
+<wire x1="-10.16" y1="-2.54" x2="-20.32" y2="-2.54" width="0.1524" layer="91"/>
+<label x="-20.32" y="-2.54" size="1.778" layer="95" rot="R180" xref="yes"/>
+</segment>
+</net>
+<net name="MOSI" class="0">
+<segment>
+<pinref part="ISP" gate="4" pin="J$1"/>
+<wire x1="99.06" y1="50.8" x2="101.6" y2="50.8" width="0.1524" layer="91"/>
+<label x="101.6" y="50.8" size="1.778" layer="95" xref="yes"/>
+</segment>
+<segment>
+<pinref part="TINY841" gate="G$1" pin="PA1"/>
+<label x="12.7" y="5.08" size="1.778" layer="95" xref="yes"/>
+<pinref part="U$1" gate="G$2" pin="J$1"/>
+<wire x1="10.16" y1="5.08" x2="45.72" y2="5.08" width="0.1524" layer="91"/>
+</segment>
+</net>

Commit message: Add files via upload
Parts:
- removed J1: CON254_2WAY, Connectors:CON254_2WAY
- removed R1, R2: 25k, rcl:R-EU_M0805
- removed R3, R4, R7, R8: 10k, rcl:R-EU_M0805
- removed U$1: CON254_8WAY, Connectors:CON254_8WAY
- added J2: CON254_18WAY3X6, Connectors:CON254_18WAY3X6
- added R10, R15, R9: 10k, RLC:R_SMD
- added R11, R14: 25k, RLC:R_SMD
- added R16: 150k, RLC:R_SMD
- ISP: value CON254_6WAY254-2X3 -> CON254_6WAY254-2X3-EDGE; device Connectors:CON254_6WAY254-2X3 -> Connectors:CON254_6WAY254-2X3-EDGE
- renumbered R5 to R12, R6 to R13
Connections:
- net GND: now also J2G$1.J$1, J2G$2.J$1, J2G$3.J$1, J2G$4.J$1, J2G$5.J$1, J2G$6.J$1, R10.P$2, R11.P$2, R12.P$2, R14.P$2, R15.P$2; no longer J1G$1.J$1, R1.1, R12.P$1, R2.1, R3.1, R7.1
- net MISO: now also J2G$7.J$1; no longer U$1G$1.J$1
- net MOSI: now also J2G$8.J$1; no longer U$1G$2.J$1
- net N$1: now also R12.P$1, R13.P$2; no longer R12.P$2, R13.P$1
- net N$10: now also J2G$9.J$1
- net N$11: now also R15.P$1, R16.P$2; no longer R7.2, R8.1
- net N$13: now also J2G$11.J$1
- net N$16: now also J2G$12.J$1; no longer U$1G$6.J$1
- net N$3: now also R14.P$1; no longer R2.2
- net N$4: now also R11.P$1; no longer R1.2
- net N$5: now also R10.P$1, R9.P$2; no longer R3.2, R4.1
- net SCK: now also J2G$10.J$1
- net V+: now also R13.P$1, R16.P$1; no longer R13.P$2, R8.2
- net VCC: now also J2G$13.J$1, J2G$14.J$1, J2G$15.J$1, J2G$16.J$1, J2G$17.J$1, J2G$18.J$1, R9.P$1; no longer J1G$2.J$1, R4.2

Commit message: Add files via upload
Parts:
- added D2: SINGLELEDKP-3216SRC-PRV, OptoElectronics:SINGLELEDKP-3216SRC-PRV
- added R1: 300, RLC:R_SMD
- added SW1: SWITCH-1P2T, Switches:SWITCH-1P2T
Connections:
- new net N$12: C6.P$1, L1.P$2, MAX5035.FB, SW1.P$1
- new net N$14: D2.A, R1.P$2
- net GND: now also D2.K
- net VCC: now also R1.P$1, SW1.P$3; no longer C6.P$1, L1.P$2, MAX5035.FB
Changed lines of the file:
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@@
 <grid distance="0.1" unitdist="inch" unit="inch" style="lines" multiple="1" display="no" altdistance="0.01" altunitdist="inch" altunit="inch"/>
 <layers>
-<layer number="1" name="Top" color="4" fill="1" visible="yes" active="no"/>
-<layer number="16" name="Bottom" color="1" fill="1" visible="yes" active="no"/>
-<layer number="17" name="Pads" color="2" fill="1" visible="yes" active="no"/>
-<layer number="18" name="Vias" color="2" fill="1" visible="yes" active="no"/>
-<layer number="19" name="Unrouted" color="6" fill="1" visible="yes" active="no"/>
-<layer number="20" name="Dimension" color="15" fill="1" visible="yes" active="no"/>
-<layer number="21" name="tPlace" color="7" fill="1" visible="yes" active="no"/>
-<layer number="22" name="bPlace" color="7" fill="1" visible="yes" active="no"/>
-<layer number="23" name="tOrigins" color="15" fill="1" visible="yes" active="no"/>
-<layer number="24" name="bOrigins" color="15" fill="1" visible="yes" active="no"/>
-<layer number="25" name="tNames" color="7" fill="1" visible="yes" active="no"/>
-<layer number="26" name="bNames" color="7" fill="1" visible="yes" active="no"/>
-<layer number="27" name="tValues" color="7" fill="1" visible="yes" active="no"/>
-<layer number="28" name="bValues" color="7" fill="1" visible="yes" active="no"/>
+<layer number="1" name="Top" color="4" fill="1" visible="no" active="no"/>
+<layer number="16" name="Bottom" color="1" fill="1" visible="no" active="no"/>
+<layer number="17" name="Pads" color="2" fill="1" visible="no" active="no"/>
+<layer number="18" name="Vias" color="2" fill="1" visible="no" active="no"/>
+<layer number="19" name="Unrouted" color="6" fill="1" visible="no" active="no"/>
+<layer number="20" name="Dimension" color="15" fill="1" visible="no" active="no"/>
+<layer number="21" name="tPlace" color="7" fill="1" visible="no" active="no"/>
+<layer number="22" name="bPlace" color="7" fill="1" visible="no" active="no"/>
+<layer number="23" name="tOrigins" color="15" fill="1" visible="no" active="no"/>
+<layer number="24" name="bOrigins" color="15" fill="1" visible="no" active="no"/>
+<layer number="25" name="tNames" color="7" fill="1" visible="no" active="no"/>
+<layer number="26" name="bNames" color="7" fill="1" visible="no" active="no"/>
+<layer number="27" name="tValues" color="7" fill="1" visible="no" active="no"/>
+<layer number="28" name="bValues" color="7" fill="1" visible="no" active="no"/>
 <layer number="29" name="tStop" color="7" fill="3" visible="no" active="no"/>
 <layer number="30" name="bStop" color="7" fill="6" visible="no" active="no"/>
@@
 <layer number="35" name="tGlue" color="7" fill="4" visible="no" active="no"/>
 <layer number="36" name="bGlue" color="7" fill="5" visible="no" active="no"/>
-<layer number="37" name="tTest" color="7" fill="1" visible="yes" active="no"/>
-<layer number="38" name="bTest" color="7" fill="1" visible="yes" active="no"/>
+<layer number="37" name="tTest" color="7" fill="1" visible="no" active="no"/>
+<layer number="38" name="bTest" color="7" fill="1" visible="no" active="no"/>
 <layer number="39" name="tKeepout" color="4" fill="11" visible="no" active="no"/>
 <layer number="40" name="bKeepout" color="1" fill="11" visible="no" active="no"/>
@@
 <layer number="44" name="Drills" color="7" fill="1" visible="no" active="no"/>
 <layer number="45" name="Holes" color="7" fill="1" visible="no" active="no"/>
-<layer number="46" name="Milling" color="3" fill="1" visible="yes" active="no"/>
-<layer number="47" name="Measures" color="7" fill="1" visible="yes" active="no"/>
-<layer number="48" name="Document" color="7" fill="1" visible="yes" active="no"/>
-<layer number="49" name="Reference" color="7" fill="1" visible="yes" active="no"/>
-<layer number="51" name="tDocu" color="7" fill="1" visible="yes" active="no"/>
-<layer number="52" name="bDocu" color="7" fill="1" visible="yes" active="no"/>
+<layer number="46" name="Milling" color="3" fill="1" visible="no" active="no"/>
+<layer number="47" name="Measures" color="7" fill="1" visible="no" active="no"/>
+<layer number="48" name="Document" color="7" fill="1" visible="no" active="no"/>
+<layer number="49" name="Reference" color="7" fill="1" visible="no" active="no"/>
+<layer number="51" name="tDocu" color="7" fill="1" visible="no" active="no"/>
+<layer number="52" name="bDocu" color="7" fill="1" visible="no" active="no"/>
 <layer number="90" name="Modules" color="5" fill="1" visible="yes" active="yes"/>
 <layer number="91" name="Nets" color="2" fill="1" visible="yes" active="yes"/>
@@
 <part name="GND17" library="supply1" deviceset="GND" device=""/>
 <part name="P+9" library="supply1" deviceset="VCC" device=""/>
+<part name="D2" library="OptoElectronics" deviceset="SINGLELED" device="KP-3216SRC-PRV"/>
+<part name="GND16" library="supply1" deviceset="GND" device=""/>
+<part name="R1" library="RLC" deviceset="R_SMD" device="" value="300"/>
+<part name="SW1" library="Switches" deviceset="SWITCH-1P2T" device=""/>
 </parts>
 <sheets>
@@
 <instance part="C5" gate="G$1" x="-63.5" y="-5.08"/>
 <instance part="L1" gate="G$1" x="-48.26" y="-12.7"/>
-<instance part="P+1" gate="VCC" x="-40.64" y="-7.62"/>
+<instance part="P+1" gate="VCC" x="-25.4" y="-7.62"/>
 <instance part="C6" gate="G$1" x="-40.64" y="-38.1"/>
 <instance part="GND11" gate="1" x="-40.64" y="-48.26"/>
@@
 <instance part="GND17" gate="1" x="-12.7" y="-83.82"/>
 <instance part="P+9" gate="VCC" x="12.7" y="-60.96"/>
+<instance part="D2" gate="G$1" x="-25.4" y="-33.02"/>
+<instance part="GND16" gate="1" x="-25.4" y="-43.18"/>
+<instance part="R1" gate="G$1" x="-25.4" y="-20.32"/>
+<instance part="SW1" gate="G$1" x="-33.02" y="-12.7"/>
 </instances>
 <busses>
@@
 <junction x="-12.7" y="-68.58"/>
 </segment>
+<segment>
+<pinref part="GND16" gate="1" pin="GND"/>
+<pinref part="D2" gate="G$1" pin="K"/>
+<wire x1="-25.4" y1="-38.1" x2="-25.4" y2="-40.64" width="0.1524" layer="91"/>
+</segment>
 </net>
 <net name="N$3" class="0">
@@
 <wire x1="-12.7" y1="22.86" x2="-12.7" y2="20.32" width="0.1524" layer="91"/>
 <junction x="-12.7" y="20.32"/>
-</segment>
-<segment>
-<pinref part="MAX5035" gate="G$1" pin="FB"/>
-<wire x1="-68.58" y1="-22.86" x2="-60.96" y2="-22.86" width="0.1524" layer="91"/>
-<wire x1="-60.96" y1="-22.86" x2="-60.96" y2="-33.02" width="0.1524" layer="91"/>
-<wire x1="-60.96" y1="-33.02" x2="-40.64" y2="-33.02" width="0.1524" layer="91"/>
-<wire x1="-40.64" y1="-33.02" x2="-40.64" y2="-12.7" width="0.1524" layer="91"/>
-<pinref part="L1" gate="G$1" pin="P$2"/>
-<wire x1="-40.64" y1="-12.7" x2="-43.18" y2="-12.7" width="0.1524" layer="91"/>
-<pinref part="P+1" gate="VCC" pin="VCC"/>
-<wire x1="-40.64" y1="-12.7" x2="-40.64" y2="-10.16" width="0.1524" layer="91"/>
-<junction x="-40.64" y="-12.7"/>
-<wire x1="-40.64" y1="-35.56" x2="-40.64" y2="-33.02" width="0.1524" layer="91"/>
-<junction x="-40.64" y="-33.02"/>
-<pinref part="C6" gate="G$1" pin="P$1"/>
 </segment>
 <segment>
@@
 <junction x="12.7" y="-76.2"/>
 </segment>
+<segment>
+<pinref part="P+1" gate="VCC" pin="VCC"/>
+<pinref part="R1" gate="G$1" pin="P$1"/>
+<wire x1="-25.4" y1="-15.24" x2="-25.4" y2="-12.7" width="0.1524" layer="91"/>
+<pinref part="SW1" gate="G$1" pin="P$3"/>
+<wire x1="-25.4" y1="-12.7" x2="-25.4" y2="-10.16" width="0.1524" layer="91"/>
+<wire x1="-27.94" y1="-12.7" x2="-25.4" y2="-12.7" width="0.1524" layer="91"/>
+<junction x="-25.4" y="-12.7"/>
+</segment>
 </net>
 <net name="IMEASURE" class="0">
@@
 </segment>
 </net>
+<net name="N$12" class="0">
+<segment>
+<pinref part="MAX5035" gate="G$1" pin="FB"/>
+<wire x1="-68.58" y1="-22.86" x2="-60.96" y2="-22.86" width="0.1524" layer="91"/>
+<wire x1="-60.96" y1="-22.86" x2="-60.96" y2="-33.02" width="0.1524" layer="91"/>
+<wire x1="-60.96" y1="-33.02" x2="-40.64" y2="-33.02" width="0.1524" layer="91"/>
+<wire x1="-40.64" y1="-33.02" x2="-40.64" y2="-12.7" width="0.1524" layer="91"/>
+<pinref part="L1" gate="G$1" pin="P$2"/>
+<wire x1="-40.64" y1="-12.7" x2="-43.18" y2="-12.7" width="0.1524" layer="91"/>
+<wire x1="-40.64" y1="-35.56" x2="-40.64" y2="-33.02" width="0.1524" layer="91"/>
+<junction x="-40.64" y="-33.02"/>
+<pinref part="C6" gate="G$1" pin="P$1"/>
+<pinref part="SW1" gate="G$1" pin="P$1"/>
+<wire x1="-38.1" y1="-12.7" x2="-40.64" y2="-12.7" width="0.1524" layer="91"/>
+<junction x="-40.64" y="-12.7"/>
+</segment>
+</net>
+<net name="N$14" class="0">
+<segment>
+<pinref part="R1" gate="G$1" pin="P$2"/>
+<pinref part="D2" gate="G$1" pin="A"/>
+<wire x1="-25.4" y1="-27.94" x2="-25.4" y2="-25.4" width="0.1524" layer="91"/>
+</segment>
+</net>

Commit message: Add files via upload
Changed lines of the file:
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@@
 <part name="V+IN2" library="supply1" deviceset="V+" device=""/>
 <part name="OP2340\" library="Semiconductors" deviceset="OPA2340" device=""/>
-<part name="P+7" library="supply1" deviceset="VCC" device=""/>
 <part name="GND15" library="supply1" deviceset="GND" device=""/>
 <part name="V+IN3" library="supply1" deviceset="V+" device=""/>
@@
 <instance part="OP2340\" gate="G$1" x="-38.1" y="45.72"/>
 <instance part="OP2340\" gate="G$2" x="25.4" y="45.72"/>
-<instance part="P+7" gate="VCC" x="15.24" y="63.5"/>
 <instance part="GND15" gate="1" x="5.08" y="30.48"/>
 <instance part="V+IN3" gate="1" x="5.08" y="66.04"/>

Commit message: Add files via upload
Parts:
- added R2, R3, R4, R5: 10k, RLC:R_SMD
- added T1: 2N7002, Semiconductors:2N7002
- added U1: L78L33A, Power:L78L33A
- renumbered OP2340\ to OP2340
Connections:
- removed net TOBLE: BLE14.UART_RX, TINY841.PA7
- new net N$17: R3.P$2, T1G$1.S, TINY841.PA7
- new net N$19: BLE14.UART_TX, R4.P$2, T1G$2.D
- new net N$21: BLE14.UART_RX, R2.P$2, T1G$1.D
- new net V3.3: BLE14.VCC, C3.P$1, R2.P$1, R4.P$1, T1G$1.G, T1G$2.G, U1.VOUT
- net GND: now also U1.GND
- net TOAT: now also R5.P$2, T1G$2.S; no longer BLE14.UART_TX
- net VCC: now also R3.P$1, R5.P$1, U1.VIN; no longer BLE14.VCC, C3.P$1
