File: hardware/VIP.sch (EAGLE design)
At the start: 38 parts, among them J2 CON254_18WAY3X6, SW1 SWITCH-1P2T, T1 2N7002, U1 L78L33A

Commit message: Add files via upload
Parts:
- renumbered BLE14 to BLE11
Connections:
- net GND: now also SW1.P$2
- net N$1: now also SW1.P$1
- net N$12: no longer SW1.P$1
- net VCC: no longer SW1.P$3
Other:
- moved on the sheet: C7, SW1
Changed lines of the file:
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@@
 <part name="GND6" library="supply1" deviceset="GND" device=""/>
 <part name="GND7" library="supply1" deviceset="GND" device=""/>
-<part name="BLE14" library="Shields" deviceset="HM-17BLE" device=""/>
+<part name="BLE11" library="Shields" deviceset="HM-17BLE" device=""/>
 <part name="C3" library="RLC" deviceset="C_SMD" device="" value="0.1uF"/>
 <part name="GND8" library="supply1" deviceset="GND" device=""/>
@@
 <instance part="GND6" gate="1" x="-12.7" y="-15.24"/>
 <instance part="GND7" gate="1" x="-22.86" y="5.08"/>
-<instance part="BLE14" gate="G$1" x="111.76" y="-17.78"/>
+<instance part="BLE11" gate="G$1" x="111.76" y="-17.78"/>
 <instance part="C3" gate="G$1" x="88.9" y="-2.54"/>
 <instance part="GND8" gate="1" x="88.9" y="-12.7"/>
@@
 <instance part="C6" gate="G$1" x="-40.64" y="-38.1"/>
 <instance part="GND11" gate="1" x="-40.64" y="-48.26"/>
-<instance part="C7" gate="G$1" x="-101.6" y="-5.08"/>
-<instance part="GND12" gate="1" x="-101.6" y="-15.24"/>
+<instance part="C7" gate="G$1" x="-106.68" y="-5.08"/>
+<instance part="GND12" gate="1" x="-106.68" y="-15.24"/>
 <instance part="D1" gate="G$1" x="-55.88" y="-17.78"/>
 <instance part="GND13" gate="1" x="-55.88" y="-27.94"/>
@@
 <instance part="GND16" gate="1" x="-25.4" y="-43.18"/>
 <instance part="R1" gate="G$1" x="-25.4" y="-20.32"/>
-<instance part="SW1" gate="G$1" x="-33.02" y="-12.7"/>
+<instance part="SW1" gate="G$1" x="-99.06" y="-22.86" rot="R270"/>
 <instance part="T1" gate="G$1" x="33.02" y="-50.8" rot="MR270"/>
 <instance part="T1" gate="G$2" x="50.8" y="-27.94" rot="MR270"/>
@@
 </segment>
 <segment>
-<pinref part="BLE14" gate="G$1" pin="GND"/>
+<pinref part="BLE11" gate="G$1" pin="GND"/>
 <pinref part="GND9" gate="1" pin="GND"/>
 <wire x1="96.52" y1="-30.48" x2="93.98" y2="-30.48" width="0.1524" layer="91"/>
@@
 <wire x1="-91.44" y1="-38.1" x2="-91.44" y2="-27.94" width="0.1524" layer="91"/>
 <pinref part="R12" gate="G$1" pin="P$2"/>
+<pinref part="SW1" gate="G$1" pin="P$2"/>
+<wire x1="-96.52" y1="-27.94" x2="-96.52" y2="-38.1" width="0.1524" layer="91"/>
+<wire x1="-96.52" y1="-38.1" x2="-91.44" y2="-38.1" width="0.1524" layer="91"/>
+<junction x="-91.44" y="-38.1"/>
 </segment>
 <segment>
@@
 <pinref part="GND12" gate="1" pin="GND"/>
 <pinref part="C7" gate="G$1" pin="P$2"/>
-<wire x1="-101.6" y1="-12.7" x2="-101.6" y2="-10.16" width="0.1524" layer="91"/>
+<wire x1="-106.68" y1="-12.7" x2="-106.68" y2="-10.16" width="0.1524" layer="91"/>
 </segment>
 <segment>
@@
 <pinref part="P+1" gate="VCC" pin="VCC"/>
 <pinref part="R1" gate="G$1" pin="P$1"/>
-<wire x1="-25.4" y1="-15.24" x2="-25.4" y2="-12.7" width="0.1524" layer="91"/>
-<pinref part="SW1" gate="G$1" pin="P$3"/>
-<wire x1="-25.4" y1="-12.7" x2="-25.4" y2="-10.16" width="0.1524" layer="91"/>
-<wire x1="-27.94" y1="-12.7" x2="-25.4" y2="-12.7" width="0.1524" layer="91"/>
-<junction x="-25.4" y="-12.7"/>
+<wire x1="-25.4" y1="-15.24" x2="-25.4" y2="-10.16" width="0.1524" layer="91"/>
 </segment>
 <segment>
@@
 <pinref part="R12" gate="G$1" pin="P$1"/>
 <pinref part="R13" gate="G$1" pin="P$2"/>
+<wire x1="-91.44" y1="-15.24" x2="-99.06" y2="-15.24" width="0.1524" layer="91"/>
+<pinref part="SW1" gate="G$1" pin="P$1"/>
+<wire x1="-99.06" y1="-15.24" x2="-99.06" y2="-17.78" width="0.1524" layer="91"/>
 </segment>
 </net>
@@
 <wire x1="-91.44" y1="0" x2="-91.44" y2="-2.54" width="0.1524" layer="91"/>
 <pinref part="C7" gate="G$1" pin="P$1"/>
-<wire x1="-101.6" y1="-2.54" x2="-101.6" y2="0" width="0.1524" layer="91"/>
-<wire x1="-101.6" y1="0" x2="-91.44" y2="0" width="0.1524" layer="91"/>
+<wire x1="-106.68" y1="-2.54" x2="-106.68" y2="0" width="0.1524" layer="91"/>
+<wire x1="-106.68" y1="0" x2="-91.44" y2="0" width="0.1524" layer="91"/>
 <junction x="-91.44" y="0"/>
 <pinref part="V+IN2" gate="1" pin="V+"/>
@@
 <junction x="-40.64" y="-33.02"/>
 <pinref part="C6" gate="G$1" pin="P$1"/>
-<pinref part="SW1" gate="G$1" pin="P$1"/>
-<wire x1="-38.1" y1="-12.7" x2="-40.64" y2="-12.7" width="0.1524" layer="91"/>
-<junction x="-40.64" y="-12.7"/>
 </segment>
 </net>
@@
 <segment>
 <wire x1="60.96" y1="-27.94" x2="60.96" y2="-20.32" width="0.1524" layer="91"/>
-<pinref part="BLE14" gate="G$1" pin="UART_TX"/>
+<pinref part="BLE11" gate="G$1" pin="UART_TX"/>
 <wire x1="96.52" y1="-20.32" x2="60.96" y2="-20.32" width="0.1524" layer="91"/>
 <pinref part="T1" gate="G$2" pin="D"/>
@@
 <wire x1="93.98" y1="2.54" x2="93.98" y2="-12.7" width="0.1524" layer="91"/>
 <junction x="88.9" y="2.54"/>
-<pinref part="BLE14" gate="G$1" pin="VCC"/>
+<pinref part="BLE11" gate="G$1" pin="VCC"/>
 <wire x1="93.98" y1="-12.7" x2="96.52" y2="-12.7" width="0.1524" layer="91"/>
 <label x="88.9" y="5.08" size="1.778" layer="95"/>
@@
 <junction x="40.64" y="-50.8"/>
 <wire x1="63.5" y1="-50.8" x2="63.5" y2="-25.4" width="0.1524" layer="91"/>
-<pinref part="BLE14" gate="G$1" pin="UART_RX"/>
+<pinref part="BLE11" gate="G$1" pin="UART_RX"/>
 <wire x1="63.5" y1="-25.4" x2="96.52" y2="-25.4" width="0.1524" layer="91"/>
 </segment>
